File: kicad PCB files./DE429_001_INSTALL.kicad_sch (KiCad schematic)
At the start: 0 parts

Commit message: Add files via upload
Parts:
- added ACC: ADXL345BCCZ-RL7, digikey-footprints:LGA-14_3x5mm_RevA, symbol dk_Motion-Sensors-Accelerometers:ADXL345BCCZ-RL7
- added AMP: LMV321, symbol Amplifier_Operational:LMV321
- added Buck: TPS54331DR, D8, symbol 2022-11-27_23-01-19:TPS54331DR
- added C1, C10, C5, C6, C8, C9: .1uF, Capacitor_SMD:C_0603_1608Metric, symbol Device:C
- added C11, C3, C4: 22uF, Capacitor_SMD:C_0603_1608Metric, symbol Device:C
- added C2: 4.7uF, Capacitor_SMD:C_0603_1608Metric, symbol Device:C
- added C7: 1uF, Capacitor_SMD:C_0603_1608Metric, symbol Device:C
- added D1, D2, D3: D_TVS, symbol Device:D_TVS
- added D1: RED_LED_Filled, symbol Device:LED_Filled
- added D4: BAT41, Diode_THT:D_DO-35_SOD27_P7.62mm_Horizontal, symbol Diode:BAT41
- added MPU: ESP32-WROOM-32D, RF_Module:ESP32-WROOM-32, symbol RF_Module:ESP32-WROOM-32D
- added PORT: USB_B_Micro, symbol Connector:USB_B_Micro
- added Power: AMS1117-3.3, Package_TO_SOT_SMD:SOT-223-3_TabPin2, symbol Regulator_Linear:AMS1117-3.3
- added Q1, Q2: MMSS8050-H-TP, digikey-footprints:SOT-23-3, symbol dk_Transistors-Bipolar-BJT-Single:MMSS8050-H-TP
- added R1, R12, R13, R5, R6, R7: 10K, Resistor_SMD:R_0603_1608Metric, symbol Device:R
- added R10: 47.5K, Resistor_SMD:R_0603_1608Metric, symbol Device:R
- added R11, R9: 2K, Resistor_SMD:R_0603_1608Metric, symbol Device:R
- added R2, R3, R4: 0R, Resistor_SMD:R_0603_1608Metric, symbol Device:R
- added R8: 22.1K, Resistor_SMD:R_0603_1608Metric, symbol Device:R
- added REF: MC14093BCP, DIP762W53P254L1848H469Q14N, symbol MC14093BCP:MC14093BCP
- added SW1, SW2: SW_Push, Button_Switch_SMD:SW_Push_SPST_NO_Alps_SKRK, symbol Switch:SW_Push
- added USB: CP2102-GMR_NRND, digikey-footprints:VFQFN-28-1EP_5x5mm, symbol dk_Interface-Controllers:CP2102-GMR_NRND
Connections:
- new net: Q1.1 (B), R5.2
- new net: Q2.1 (B), R6.2
- new net: R7.2, USB.11 (SUSPEND)
- new net: C1.2, C2.2, USB.6 (VDD), USB.7 (REGIN)
- new net: R10.2, R8.2, USB.8 (VBUS)
- new net: R9.1, USB.9 (RST)
- new net: C6.2, MPU.3 (EN), R1.2
- new net: C11.1, Power.2 (VO)
- new net: MPU.34 (RXD0/IO3), R4.1
- new net: MPU.35 (TXD0/IO1), R3.1
- new net: D1.2 (A2), D4.2 (A), PORT.1 (VBUS)
- new net: D1.2 (A), R11.1
- new net: AMP.3 (-), R12.2, R13.1
- new net: ACC.6 (VS), C7.2
- new net 3V3: ACC.1 (VDD_I/O), AMP.2 (V-), C4.1, C5.1, C7.1, C8.2, MPU.2 (VDD), R1.1, R9.2
- new net EN: C10.2, Q1.3 (C), SW2.2
- new net EXT_5V: C3.1, D4.1 (K), Power.3 (VI), R11.2
- new net GND: ACC.2 (GND), AMP.5 (V+), C1.1, C10.1, C11.2, C2.1, C3.2, C4.2, C5.2, C6.1, C8.1, C9.1, D1.1 (A1), D1.1 (K), D2.1 (A1), D3.1 (A1), MPU.1 (GND), MPU.15 (GND), MPU.38 (GND), MPU.39 (GND), PORT.5 (GND), Power.1 (GND), Q2.2 (E), R10.1, R2.1, R5.1, R7.1, SW1.1, SW2.1, USB.28 (DTR), USB.3 (GND)
- new net GND-A: R2.2
- new net IO0: C9.2, Q2.3 (C), SW1.2
- new net RTS: Q1.2 (E), R6.1, USB.24 (RTS)
- new net RXD: R4.2, USB.25 (RXD)
- new net SCL: ACC.13 (SDA), MPU.36 (IO22)
- new net SDA: ACC.14 (SCL), MPU.33 (IO21)
- new net SDO: ACC.12 (SDO), MPU.21 (SDO/SD0)
- new net TXD: R3.2, USB.26 (TXD)
- new net USB-DP: D3.2 (A2), PORT.2 (D-), USB.5 (D-)
- new net USB_DN: D2.2 (A2), PORT.3 (D+), USB.4 (D+)
- new net VBUS: AMP.4, R13.2, R8.1
- no-connect marks 0 -> 3
